File: PCI Design/Soletrando-e-Aprendendo_v1.kicad_sch (KiCad schematic)
At the start: 45 parts, among them J1 I2C_Con, J2 I2C_Con, J3 I2C_Con, Q1 BC817, Q2 IRF9540N, SW1 Botão_A, SW2 Botão_B, SW3 ON/OFF, SW4 Cancel, SW5 Config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

Commit message: Adicionando novos capacitores no circuito
Parts:
- added C10, C11, C12, C7, C9: 100nF, Capacitor_SMD:C_0805_2012Metric, symbol Device:C
- added C13: 10uF, Capacitor_SMD:CP_Elec_5x5.4, symbol Device:C_Polarized
- added C14: 10uF/16V, Capacitor_SMD:CP_Elec_5x5.4, symbol Device:C_Polarized
- added C8: 100uF/16V, Capacitor_THT:CP_Radial_D5.0mm_P2.50mm, symbol Device:C_Polarized
- added R7: 10K, Resistor_SMD:R_0805_2012Metric, symbol Device:R
- C2: value 10uF/25V -> 10uF/16V
- C6: value 220uF/16V -> 470uF/16V
Connections:
- net +3V3: now also C10.1, C11.1, C12.1, C7.1, C8.1, C9.1
- net +5V: now also C13.1, C14.1
- net GNDREF: now also C10.2, C11.2, C12.2, C13.2, C14.2, C7.2, C8.2, C9.2, R7.2
- net at Q1.1 (B), R1.2: now also R7.1
Other:
- moved on the sheet: BZ1, BZ2, D2, J1, J2, J3, Q1, R1, R4, R5, R6, SW1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
