File: PCI Design/Soletrando-e-Aprendendo_v1.kicad_pcb (KiCad board)
At the start: 2 copper layers, 115 x 115 mm, 57 parts, among them J1 I2C_Con, J2 I2C_Con, J3 I2C_Con, Q1 BC817, Q2 IRF9540N, SW1 Botão_A, SW2 Botão_B, SW3 ON/OFF, SW4 Cancel, SW5 Config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

Commit message: Adicionando plano GND ao TopOverLayer
Routing:
- added copper zone on F.Cu, net GNDREF
Changed lines of the file:
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@@
 	)
 	(gr_text "Grupo de Pesquisa INOVA Pecém"
-		(at 118 146.9 0)
+		(at 118 146.6 0)
 		(layer "F.SilkS")
 		(effects
@@
 		(net 2)
 		(net_name "GNDREF")
-		(layer "B.Cu")
+		(layers "F.Cu" "B.Cu")
 		(name "PLANO-GND")
 		(hatch edge 0.5)
@@
 		(members "0a0a690c-318b-47e6-abf4-9050ac319c09" "fc459292-57a0-4b8c-8709-5125f7e50b55")
 	)
+	(group ""
+		(members "25687445-14ac-46d8-bae8-b64c5b2e4593")
+	)
 	(embedded_fonts no)
